File: redroid_go.kicad_pcb (KiCad board)
At the start: 2 copper layers, 70 x 95 mm, 100 parts, among them J1 USB4105-GF-A, J2 5051101892, J3 Conn_01x02_Pin, J4 Conn_01x10_Pin, Q1 UMH3N, Q2 PMOS, Q3 UMH3N, SW1 UP, SW10 A, SW11 SW_SPDT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

Commit message: Minor fix in via
Routing:
- net IO14: track 39.3 -> 37.4 mm
Changed lines of the file:
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@@
 	)
 	(segment
-		(start 178.5 77.5)
-		(end 171.25 77.5)
+		(start 174.5 77)
+		(end 170.75 80.75)
+		(width 0.2)
+		(layer "F.Cu")
+		(net 51)
+	)
+	(segment
+		(start 178.5 77)
+		(end 174.5 77)
 		(width 0.2)
 		(layer "F.Cu")
@@
 	)
 	(via
-		(at 178.5 77.5)
+		(at 178.5 77)
 		(size 0.6)
 		(drill 0.3)
@@
 	)
 	(via
-		(at 171.25 77.5)
+		(at 170.75 80.75)
 		(size 0.6)
 		(drill 0.3)
@@
 	)
 	(segment
-		(start 179.75 77.5)
-		(end 178.5 77.5)
+		(start 170.75 80.75)
+		(end 168.5 83)
 		(width 0.2)
 		(layer "B.Cu")
@@
 	)
 	(segment
-		(start 168.5 84.67)
-		(end 168.5 83.5)
-		(width 0.2)
-		(layer "B.Cu")
-		(net 51)
-	)
-	(segment
-		(start 171.25 80.75)
-		(end 171.25 77.5)
+		(start 179.75 77)
+		(end 179.75 76.5)
 		(width 0.2)
 		(layer "B.Cu")
@@
 	)
 	(segment
-		(start 179.75 76.5)
-		(end 179.75 77.5)
+		(start 178.5 77)
+		(end 179.75 77)
 		(width 0.2)
 		(layer "B.Cu")
@@
 	)
 	(segment
-		(start 168.5 83.5)
-		(end 171.25 80.75)
+		(start 168.5 83)
+		(end 168.5 84.67)
 		(width 0.2)
 		(layer "B.Cu")
