File: pcb/redroid_go.kicad_sch (KiCad schematic)
At the start: 100 parts, among them J1 USB4105-GF-A, J2 5051101892, J3 Conn_01x02_Pin, J4 Conn_01x10_Pin, Q1 UMH3N, Q2 PMOS, Q3 UMH3N, SW1 UP, SW10 A, SW11 SW_SPDT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

Commit message: Add missing GND connectio to ESP32
Connections:
- net GND: now also U1.15 (GND)
Changed lines of the file:
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@@
 	)
 	(junction
+		(at 67.31 76.2)
+		(diameter 0)
+		(color 0 0 0 0)
+	)
+	(junction
 		(at 180.34 21.59)
 		(diameter 0)
@@
 	(wire
 		(pts
-			(xy 67.31 40.64) (xy 67.31 109.22)
+			(xy 67.31 40.64) (xy 67.31 76.2)
 		)
 		(stroke
@@
 	(wire
 		(pts
+			(xy 67.31 76.2) (xy 67.31 109.22)
+		)
+		(stroke
+			(width 0)
+			(type default)
+		)
+	)
+	(wire
+		(pts
 			(xy 359.41 151.13) (xy 359.41 179.07)
 		)
@@
 		)
 		(stroke
+			(width 0)
+			(type default)
+		)
+	)
+	(wire
+		(pts
+			(xy 67.31 76.2) (xy 71.12 76.2)
+		)
+		(stroke

Commit message: Change switch connection to improve PCB
Connections:
- net at C2.1, F1.2, TP2.1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: now also SW11.3 (C); no longer SW11.2 (B)
- net at U3.8 (EN): now also SW11.2 (B); no longer SW11.1 (A)
Other:
- moved on the sheet: SW11
Changed lines of the file:
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@@
 	(wire
 		(pts
-			(xy 350.52 30.48) (xy 350.52 43.18)
-		)
-		(stroke
-			(width 0)
-			(type default)
-		)
-	)
-	(wire
-		(pts
 			(xy 153.67 238.76) (xy 160.02 238.76)
 		)
@@
 	(wire
 		(pts
+			(xy 290.83 30.48) (xy 290.83 45.72)
+		)
+		(stroke
+			(width 0)
+			(type default)
+		)
+	)
+	(wire
+		(pts
 			(xy 269.24 227.33) (xy 271.78 227.33)
 		)
@@
 	(wire
 		(pts
-			(xy 293.37 33.02) (xy 290.83 33.02)
-		)
-		(stroke
-			(width 0)
-			(type default)
-		)
-	)
-	(wire
-		(pts
 			(xy 219.71 180.34) (xy 219.71 191.77)
 		)
@@
 	(wire
 		(pts
+			(xy 350.52 27.94) (xy 350.52 43.18)
+		)
+		(stroke
+			(width 0)
+			(type default)
+		)
+	)
+	(wire
+		(pts
 			(xy 356.87 60.96) (xy 359.41 60.96)
 		)
@@
 	(wire
 		(pts
+			(xy 312.42 27.94) (xy 350.52 27.94)
+		)
+		(stroke
+			(width 0)
+			(type default)
+		)
+	)
+	(wire
+		(pts
 			(xy 93.98 170.18) (xy 96.52 170.18)
 		)
@@
 	(wire
 		(pts
-			(xy 303.53 30.48) (xy 350.52 30.48)
-		)
-		(stroke
-			(width 0)
-			(type default)
-		)
-	)
-	(wire
-		(pts
 			(xy 354.33 71.12) (xy 359.41 71.12)
 		)
@@
 	(wire
 		(pts
+			(xy 290.83 30.48) (xy 302.26 30.48)
+		)
+		(stroke
+			(width 0)
+			(type default)
+		)
+	)
+	(wire
+		(pts
 			(xy 83.82 218.44) (xy 83.82 241.3)
 		)
@@
 	(wire
 		(pts
-			(xy 290.83 33.02) (xy 290.83 45.72)
-		)
-		(stroke
-			(width 0)
-			(type default)
-		)
-	)
-	(wire
-		(pts
 			(xy 213.36 87.63) (xy 217.17 87.63)
 		)
@@
 	(symbol
 		(lib_id "Switch:SW_SPDT")
-		(at 298.45 33.02 0)
+		(at 307.34 27.94 0)
+		(mirror y)
 		(unit 1)
 		(exclude_from_sim no)
@@
 		(on_board yes)
 		(dnp no)
-		(fields_autoplaced yes)
 		(property "Reference" "SW11"
-			(at 298.45 24.13 0)
+			(at 307.34 19.05 0)
 			(effects
 				(font
@@
 		)
 		(property "Value" "SW_SPDT"
-			(at 298.45 26.67 0)
+			(at 307.34 21.59 0)
 			(effects
 				(font
@@
 		)
 		(property "Footprint" "MK-12F03-G015:MK-12F03-G015"
-			(at 298.45 33.02 0)
+			(at 307.34 27.94 0)
 			(effects
 				(font
@@
 		)
 		(property "Datasheet" "~"
-			(at 298.45 40.64 0)
+			(at 307.34 35.56 0)
 			(effects
 				(font
@@
 		)
 		(property "Description" "Switch, single pole double throw"
-			(at 298.45 33.02 0)
+			(at 307.34 27.94 0)
 			(effects
 				(font

Commit message: Add missing value for some components
Parts:
- PAM8304: value ~ -> PAM8304
- U6: value ~ -> uSD
Changed lines of the file:
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@@
 			)
 		)
-		(property "Value" "~"
+		(property "Value" "uSD"
 			(at 248.92 248.92 0)
 			(effects
@@
 			)
 		)
-		(property "Value" "~"
+		(property "Value" "PAM8304"
 			(at 69.85 212.09 0)
 			(effects
