File: pcb/redroid_go.kicad_sch (KiCad schematic)
At the start: 100 parts, among them J1 USB4105-GF-A, J2 5051101892, J3 Conn_01x02_Pin, J4 Conn_01x10_Pin, Q1 UMH3N, Q2 PMOS, Q3 UMH3N, SW1 UP, SW10 A, SW11 SW_SPDT, SW2 DOWN, SW3 LEFT, SW4 RIGHT, SW5 MENU, SW6 VOLUME, SW7 SELECT, SW8 START, SW9 B, U1 ESP32-WROVER-E-N16R8, U2 CH340C, U3 MP2161GJ-Z, U4 XC6802A42XMR-G, U5 XC6206PxxxMR, U6 uSD, U7 NC7SZ125M5X, U8 NC7SZ125M5X, U9 NC7SZ125M5X

Commit message: Fix Q2 polarity
Connections:
- net VBAT: now also Q2.1 (D); no longer Q2.3 (S)
- net at D1.1 (K), F1.1: now also Q2.3 (S); no longer Q2.1 (D)
Changed lines of the file:
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@@
 	)
 	(junction
-		(at 127 151.13)
+		(at 279.4 45.72)
 		(diameter 0)
 		(color 0 0 0 0)
 	)
 	(junction
-		(at 55.88 223.52)
+		(at 127 151.13)
 		(diameter 0)
 		(color 0 0 0 0)
 	)
 	(junction
-		(at 279.4 45.72)
+		(at 55.88 223.52)
 		(diameter 0)
 		(color 0 0 0 0)
@@
 	(wire
 		(pts
-			(xy 279.4 45.72) (xy 281.94 45.72)
+			(xy 276.86 45.72) (xy 279.4 45.72)
 		)
 		(stroke
@@
 	(wire
 		(pts
-			(xy 276.86 45.72) (xy 279.4 45.72)
-		)
-		(stroke
-			(width 0)
-			(type default)
-		)
-	)
-	(wire
-		(pts
 			(xy 370.84 97.79) (xy 370.84 93.98)
 		)
@@
 	(wire
 		(pts
-			(xy 279.4 26.67) (xy 279.4 30.48)
-		)
-		(stroke
-			(width 0)
-			(type default)
-		)
-	)
-	(wire
-		(pts
 			(xy 246.38 228.6) (xy 251.46 228.6)
 		)
@@
 	(wire
 		(pts
+			(xy 279.4 40.64) (xy 279.4 45.72)
+		)
+		(stroke
+			(width 0)
+			(type default)
+		)
+	)
+	(wire
+		(pts
 			(xy 119.38 227.33) (xy 123.19 227.33)
 		)
@@
 	(wire
 		(pts
-			(xy 279.4 40.64) (xy 279.4 45.72)
-		)
-		(stroke
-			(width 0)
-			(type default)
-		)
-	)
-	(wire
-		(pts
 			(xy 314.96 181.61) (xy 313.69 181.61)
 		)
@@
 	(wire
 		(pts
+			(xy 279.4 45.72) (xy 281.94 45.72)
+		)
+		(stroke
+			(width 0)
+			(type default)
+		)
+	)
+	(wire
+		(pts
 			(xy 109.22 135.89) (xy 109.22 144.78)
 		)
@@
 	(wire
 		(pts
+			(xy 279.4 26.67) (xy 279.4 30.48)
+		)
+		(stroke
+			(width 0)
+			(type default)
+		)
+	)
+	(wire
+		(pts
 			(xy 180.34 67.31) (xy 200.66 67.31)
 		)
@@
 		(lib_id "Simulation_SPICE:PMOS")
 		(at 276.86 35.56 0)
-		(mirror x)
 		(unit 1)
 		(body_style 1)
@@
 		(dnp no)
 		(property "Reference" "Q2"
-			(at 283.21 36.8301 0)
+			(at 283.21 34.2899 0)
 			(show_name no)
 			(do_not_autoplace no)
@@
 		)
 		(property "Value" "PMOS"
-			(at 283.21 34.2901 0)
+			(at 283.21 36.8299 0)
 			(show_name no)
 			(do_not_autoplace no)
@@
 		)
 		(property "Footprint" "Package_TO_SOT_SMD:SOT-23"
-			(at 281.94 38.1 0)
+			(at 281.94 33.02 0)
 			(hide yes)
 			(show_name no)
@@
 		)
 		(property "Datasheet" "https://ngspice.sourceforge.io/docs/ngspice-html-manual/manual.xhtml#cha_MOSFETs"
-			(at 276.86 22.86 0)
+			(at 276.86 48.26 0)
 			(hide yes)
 			(show_name no)
@@
 		)
 		(property "Sim.Device" "PMOS"
-			(at 276.86 18.415 0)
+			(at 276.86 52.705 0)
 			(hide yes)
 			(show_name no)
@@
 		)
 		(property "Sim.Type" "VDMOS"
-			(at 276.86 16.51 0)
+			(at 276.86 54.61 0)
 			(hide yes)
 			(show_name no)
@@
 		)
 		(property "Sim.Pins" "1=D 2=G 3=S"
-			(at 276.86 20.32 0)
+			(at 276.86 50.8 0)
 			(hide yes)
 			(show_name no)
